Commit message: [fix bug] fix robot description: urdf model and spawn

File: robot_description/urdf/caterpillar_mobile_robot.urdf (robot description, URDF)
Before this commit: robot my_robot, 4 links, 3 joints
Links:
- link head: geometry visual box size=0.05 0.1 0.03
- link leg2: geometry visual box size=0.3 0.05 0.12
Joints:
- joint leg1connect: origin xyz=0 .125 0.06 -> xyz=0 0.125 0.06
- joint leg2connect: origin xyz=0 -.125 0.06 -> xyz=0 -0.125 0.06

Commit message: [feature] change model from own to turtlebot3 burger

File: robot_description/urdf/caterpillar_mobile_robot.urdf (robot description, URDF)
Before this commit: robot caterpillar_mobile_robot, 4 links, 3 joints
Links:
- link base_link: mass 5 -> None; geometry collision box size=0.25 0.2 0.05; visual box size=0.25 0.2 0.05
- link head: mass None -> 5; geometry collision box size=0.05 0.1 0.03; visual box size=0.05 0.1 0.03
- link leg1: geometry collision box size=0.30 0.05 0.12; visual box size=0.30 0.05 0.12
- link leg2: geometry collision box size=0.3 0.05 0.12; visual box size=0.3 0.05 0.12
