Commit message: [software] few fixes in gazebo spawn/server

File: robot_description/urdf/tracked_robot.urdf.xacro (robot description, xacro)
@@ -1,5 +1,10 @@
 <?xml version="1.0"?>
-<!-- The caterpillar mobile robot model-->
-<robot name="caterpillar_mobile_robot" xmlns:xacro="http://www.ros.org/wiki/xacro">
+<robot name="tracked_robot" xmlns:xacro="http://www.ros.org/wiki/xacro">
+  <link name="base_footprint"/>
+  <joint name="base_joint" type="fixed">
+    <parent link="base_footprint"/>
+    <child link="base_link"/>
+    <origin xyz="0.0 0.0 0.010" rpy="0 0 0"/>
+  </joint>
   <link name="base_link">
     <visual>

Commit message: [software] add model for a wheeled robot

File: robot_description/urdf/tracked_robot.urdf.xacro (robot description, xacro)
@@ -1,93 +1,338 @@
 <?xml version="1.0"?>
 <robot name="tracked_robot" xmlns:xacro="http://www.ros.org/wiki/xacro">
+  <xacro:include filename="$(find robot_description)/urdf/inertial_macros.xacro"/>
+  <xacro:include filename="$(find robot_description)/urdf/common_properties.xacro"/>
+  <xacro:arg name="laser_visual" default="true"/>
+  <xacro:property name="ROBOT_LENGTH"     value="0.30" />
+  <xacro:property name="ROBOT_WIDTH"      value="0.30" />
+  <xacro:property name="ROBOT_HEIGHT"     value="0.28" />
+  <xacro:property name="TRACK_LENGTH"     value="0.30" />
+  <xacro:property name="TRACK_WIDTH"      value="0.05" />
+  <xacro:property name="TRACK_HEIGHT"     value="0.15" />
+  <xacro:property name="TRACK_SEPARATION" value="0.23" />
+  <xacro:property name="WHEEL_RADIUS"     value="0.04" />
+  <xacro:property name="WHEEL_WIDTH"      value="0.025" />
+  <xacro:property name="WHEEL_MASS"       value="0.1" />
+  <xacro:property name="BASE_LENGTH"      value="0.22" />
+  <xacro:property name="BASE_WIDTH"       value="0.20" />
+  <xacro:property name="BASE_HEIGHT"      value="0.03" />
+  <xacro:property name="BASE_MASS"        value="1" />
   <link name="base_footprint"/>
+  <link name="base_link">
+    <visual>
+      <origin xyz="0 0 ${2.5*WHEEL_RADIUS}" />
+      <geometry>
+        <box size="${BASE_LENGTH} ${BASE_WIDTH} ${BASE_HEIGHT}"/>
+      </geometry>
+      <material name="grey"/>
+    </visual>
+    <collision>
+      <origin xyz="0 0 ${2.5*WHEEL_RADIUS}" rpy="0 0 0"/>
+      <geometry>
+        <box size="${BASE_LENGTH} ${BASE_WIDTH} ${BASE_HEIGHT}"/>
+      </geometry>
+    </collision>
+    <xacro:solid_cuboid_inertial
+      length="${BASE_LENGTH}" width="${BASE_WIDTH}" height="${BASE_HEIGHT}" mass="${BASE_MASS}">
+      <origin xyz="0 0 ${2.5*WHEEL_RADIUS}" rpy="0 0 0"/>
+    </xacro:solid_cuboid_inertial>
+  </link>
   <joint name="base_joint" type="fixed">
     <parent link="base_footprint"/>
     <child link="base_link"/>
-    <origin xyz="0.0 0.0 0.010" rpy="0 0 0"/>
-  </joint>
-  <link name="base_link">
-    <visual>
-      <origin xyz="0 0 0.1" />
-      <geometry>
-        <box size="0.25 0.2 0.05"/>
-      </geometry>
-      <material name="gray">
-        <color rgba="0.2 0.2 0.2 1" />
+    <origin xyz="0 0 0" rpy="0 0 0"/>
+  </joint>
+  <gazebo reference="base_link">
+    <material>Gazebo/Grey</material>
+    <turnGravityOff>false</turnGravityOff>
+    <selfCollide>false</selfCollide>
+  </gazebo>
+  <link name="back_left_wheel">
+    <visual>
+      <origin xyz="0 0 0"/>
+      <geometry>
+        <cylinder radius="${WHEEL_RADIUS}" length="${WHEEL_WIDTH}" />
+      </geometry>
+      <material name="grey"/>
+    </visual>
+    <collision>
+      <origin xyz="0 0 0"/>
+      <geometry>
+        <cylinder radius="${WHEEL_RADIUS}" length="${WHEEL_WIDTH}" />
+      </geometry>
+    </collision>
+    <xacro:solid_cylinder_inertial r="${WHEEL_RADIUS}" h="${WHEEL_WIDTH}" mass="${WHEEL_MASS}" >
+      <origin xyz="0 0 0" rpy="0 0 0" />
+    </xacro:solid_cylinder_inertial>
+  </link>
+  <joint name="back_left_wheel_connect" type="continuous">
+    <parent link="base_link"/>
+    <child link="back_left_wheel"/>
+    <origin xyz="${WHEEL_RADIUS - ROBOT_LENGTH/2} 0.125 0.06" rpy="-1.57 0 0"/>
+    <axis xyz="0 0 1"/>
+  </joint>
+  <gazebo reference="back_left_wheel">
+    <material>Gazebo/Grey</material>
+    <turnGravityOff>false</turnGravityOff>
+    <selfCollide>false</selfCollide>
+  </gazebo>
+  <link name="back_right_wheel">
+    <visual>
+      <origin xyz="0 0 0"/>
+      <geometry>
+        <cylinder radius="${WHEEL_RADIUS}" length="${WHEEL_WIDTH}" />
+      </geometry>
+      <material name="grey"/>
+    </visual>
+    <collision>
+      <origin xyz="0 0 0"/>
+      <geometry>
+        <cylinder radius="${WHEEL_RADIUS}" length="${WHEEL_WIDTH}" />
+      </geometry>
+    </collision>
+    <xacro:solid_cylinder_inertial r="${WHEEL_RADIUS}" h="${WHEEL_WIDTH}" mass="${WHEEL_MASS}" >
+      <origin xyz="0 0 0" rpy="0 0 0" />
+    </xacro:solid_cylinder_inertial>
+  </link>
+  <joint name="back_right_wheel_connect" type="continuous">
+    <parent link="base_link"/>
+    <child link="back_right_wheel"/>
+    <origin xyz="${WHEEL_RADIUS - ROBOT_LENGTH/2} -0.125 0.06" rpy="-1.57 0 0"/>
+    <axis xyz="0 0 1"/>
+  </joint>
+  <gazebo reference="back_right_wheel">
+    <material>Gazebo/Grey</material>
+    <turnGravityOff>false</turnGravityOff>
+    <selfCollide>false</selfCollide>
+  </gazebo>
+  <link name="mid_left_wheel">
+    <visual>
+      <origin xyz="0 0 0"/>
+      <geometry>
+        <cylinder radius="${WHEEL_RADIUS}" length="${WHEEL_WIDTH}" />
+      </geometry>
+      <material name="grey"/>
+    </visual>
+    <collision>
+      <origin xyz="0 0 0"/>
+      <geometry>
+        <cylinder radius="${WHEEL_RADIUS+0.0001}" length="${WHEEL_WIDTH}" />
+      </geometry>
+    </collision>
+    <xacro:solid_cylinder_inertial r="${WHEEL_RADIUS}" h="${WHEEL_WIDTH}" mass="${WHEEL_MASS}" >
+      <origin xyz="0 0 0" rpy="0 0 0" />
+    </xacro:solid_cylinder_inertial>
+  </link>
+  <joint name="mid_left_wheel_connect" type="continuous">
+    <parent link="base_link"/>
+    <child link="mid_left_wheel"/>
+    <origin xyz="0 0.125 0.06" rpy="-1.57 0 0"/>
+    <axis xyz="0 0 1"/>
+  </joint>
+  <gazebo reference="mid_left_wheel">
+    <material>Gazebo/Grey</material>
+    <turnGravityOff>false</turnGravityOff>
+    <selfCollide>false</selfCollide>
+  </gazebo>
+  <link name="mid_right_wheel">
+    <visual>
+      <origin xyz="0 0 0"/>
+      <geometry>
+        <cylinder radius="${WHEEL_RADIUS}" length="${WHEEL_WIDTH}" />
+      </geometry>
+      <material name="grey"/>
+    </visual>
+    <collision>
+      <origin xyz="0 0 0"/>
+      <geometry>
+        <cylinder radius="${WHEEL_RADIUS+0.0001}" length="${WHEEL_WIDTH}" />
+      </geometry>
+    </collision>
+    <xacro:solid_cylinder_inertial r="${WHEEL_RADIUS}" h="${WHEEL_WIDTH}" mass="${WHEEL_MASS}" >
+      <origin xyz="0 0 0" rpy="0 0 0" />
+    </xacro:solid_cylinder_inertial>
+  </link>
+  <joint name="mid_right_wheel_connect" type="continuous">
+    <parent link="base_link"/>
+    <child link="mid_right_wheel"/>
+    <origin xyz="0 -0.125 0.06" rpy="-1.57 0 0"/>
+    <axis xyz="0 0 1"/>
+  </joint>
+  <gazebo reference="mid_right_wheel">
+    <material>Gazebo/Grey</material>
+    <turnGravityOff>false</turnGravityOff>
+    <selfCollide>false</selfCollide>
+  </gazebo>
+  <link name="front_left_wheel">
+    <visual>
+      <origin xyz="0 0 0"/>
+      <geometry>
+        <cylinder radius="${WHEEL_RADIUS}" length="${WHEEL_WIDTH}" />
+      </geometry>
+      <material name="grey"/>
+    </visual>
+    <collision>
+      <origin xyz="0 0 0"/>
+      <geometry>
+        <cylinder radius="${WHEEL_RADIUS}" length="${WHEEL_WIDTH}" />
+      </geometry>
+    </collision>
+    <xacro:solid_cylinder_inertial r="${WHEEL_RADIUS}" h="${WHEEL_WIDTH}" mass="${WHEEL_MASS}" >
+      <origin xyz="0 0 0" rpy="0 0 0" />
+    </xacro:solid_cylinder_inertial>
+  </link>
+  <joint name="front_left_wheel_connect" type="continuous">
+    <parent link="base_link"/>
+    <child link="front_left_wheel"/>
+    <origin xyz="${ROBOT_LENGTH/2 - WHEEL_RADIUS} 0.125 0.06" rpy="-1.57 0 0"/>
+    <axis xyz="0 0 1"/>
+  </joint>
+  <gazebo reference="front_left_wheel">
+    <material>Gazebo/Grey</material>
+    <turnGravityOff>false</turnGravityOff>
+    <selfCollide>false</selfCollide>
+  </gazebo>
+  <link name="front_right_wheel">
+    <visual>
+      <origin xyz="0 0 0"/>
+      <geometry>
+        <cylinder radius="${WHEEL_RADIUS}" length="${WHEEL_WIDTH}" />
+      </geometry>
+      <material name="grey"/>
+    </visual>
+    <collision>
+      <origin xyz="0 0 0"/>
+      <geometry>
+        <cylinder radius="${WHEEL_RADIUS}" length="${WHEEL_WIDTH}" />
+      </geometry>
+    </collision>
+    <xacro:solid_cylinder_inertial r="${WHEEL_RADIUS}" h="${WHEEL_WIDTH}" mass="${WHEEL_MASS}" >
+      <origin xyz="0 0 0" rpy="0 0 0" />
+    </xacro:solid_cylinder_inertial>
+  </link>
+  <joint name="front_right_wheel_connect" type="continuous">
+    <parent link="base_link"/>
+    <child link="front_right_wheel"/>
+    <origin xyz="${ROBOT_LENGTH/2 - WHEEL_RADIUS} -0.125 0.06" rpy="-1.57 0 0"/>
+    <axis xyz="0 0 1"/>
+  </joint>
+  <gazebo reference="front_right_wheel">
+    <material>Gazebo/Grey</material>
+    <turnGravityOff>false</turnGravityOff>
+    <selfCollide>false</selfCollide>
+  </gazebo>
+  <link name="head">
+    <visual>
+      <origin xyz="0 0 0" />
+      <geometry>
+        <box size="${BASE_LENGTH} 0.24 0.10" />
+      </geometry>
+      <material name="black">
+        <color rgba="0 0 0 1"/>
       </material>
     </visual>
     <collision>
       <geometry>
-        <box size="0.25 0.2 0.05"/>
-      </geometry>
-    </collision>
-  </link>
-  <link name="leg1">
-    <visual>
-      <origin xyz="0 0 0" />
-      <geometry>
-        <box size="0.30 0.05 0.12" />
-      </geometry>
-      <material name="gray2">
-        <color rgba="0.28 0.34 0.39 1"/>
+        <box size="${BASE_LENGTH} 0.24 0.10"/>
+      </geometry>
+    </collision>
+    <xacro:solid_cuboid_inertial
+      length="${BASE_LENGTH}" width="0.24" height="0.10" mass="0.01">
+      <origin xyz="0 0 0" rpy="0 0 0"/>
+    </xacro:solid_cuboid_inertial>
+  </link>
+  <joint name="head_connect" type="fixed">
+    <origin xyz="0 0 0.165" />
+    <parent link="base_link"/>
+    <child link="head"/>
+  </joint>
+  <gazebo reference="head">
+    <material>Gazebo/Black</material>
+    <turnGravityOff>false</turnGravityOff>
+    <selfCollide>false</selfCollide>
+  </gazebo>
+  <link name="base_scan">
+    <visual>
+      <origin xyz="0 0 0"/>
+      <geometry>
+        <box size="0.02 0.02 0.02" />
+      </geometry>
+      <material name="blue">
+        <color rgba="0 1 0 1"/>
       </material>
     </visual>
-    <collision>
-      <geometry>
-        <box size="0.30 0.05 0.12"/>
-      </geometry>
-    </collision>
-  </link>
-  <joint name="leg1connect" type="fixed">
-    <origin xyz="0 0.125 0.06" />
-    <parent link="base_link"/>
-    <child link="leg1"/>
-  </joint>
-  <link name="leg2">
-    <visual>
-      <origin xyz="0 0 0" />
-      <geometry>
-        <box size="0.3 0.05 0.12" />
-      </geometry>
-      <material name="gray3">
-        <color rgba="0.15 0.22 0.27 1"/>
-      </material>
-    </visual>
-    <collision>
-      <geometry>
-        <box size="0.3 0.05 0.12"/>
-      </geometry>
-    </collision>
-  </link>
-  <joint name="leg2connect" type="fixed">
-    <origin xyz="0 -0.125 0.06" />
-    <parent link="base_link"/>
-    <child link="leg2"/>
-  </joint>
-  <link name="head">
-    <visual>
-      <origin xyz="0 0 0" />
-      <geometry>
-        <box size="0.05 0.1 0.03" />
-      </geometry>
-      <material name="red">
-        <color rgba="0.7 0 0 1"/>
-      </material>
-    </visual>
-    <inertial>
-      <mass value="5"/>
-      <origin xyz="0 0 0.1" rpy="0 0 0"/>
-      <inertia ixx="0.0395416666667" ixy="0" ixz="0" iyy="0.106208333333" iyz="0" izz="0.106208333333"/>
-    </inertial>
-    <collision>
-      <geometry>
-        <box size="0.05 0.1 0.03"/>
-      </geometry>
-    </collision>
-  </link>
-  <joint name="head_connect" type="fixed">
-    <origin xyz="0.10 0 0.135" />
-    <parent link="base_link"/>
-    <child link="head"/>
-  </joint>
+    <xacro:solid_cuboid_inertial
+      length="0.02" width="0.02" height="0.02" mass="0.1">
+      <origin xyz="0 0 0" rpy="0 0 0"/>
+    </xacro:solid_cuboid_inertial>
+    <collision>
+      <geometry>
+        <box size="0.02 0.02 0.02"/>
+      </geometry>
+    </collision>
+  </link>
+  <joint name="base_scan_connect" type="fixed">
+    <origin xyz="0 0 0.06" />
+    <parent link="head"/>
+    <child link="base_scan"/>
+  </joint>
+  <gazebo reference="base_scan">
+    <material>Gazebo/White</material>
+    <turnGravityOff>false</turnGravityOff>
+    <selfCollide>false</selfCollide>
+  </gazebo>
+  <gazebo>
+    <plugin name="tracked_robot_controller" filename="libgazebo_ros_diff_drive.so">
+      <commandTopic>cmd_vel</commandTopic>
+      <odometryTopic>odom</odometryTopic>
+      <odometryFrame>odom</odometryFrame>
+      <odometrySource>world</odometrySource>
+      <publishOdomTF>true</publishOdomTF>
+      <robotBaseFrame>base_footprint</robotBaseFrame>
+      <publishWheelTF>false</publishWheelTF>
+      <publishTf>true</publishTf>
+      <publishWheelJointState>true</publishWheelJointState>
+      <legacyMode>true</legacyMode>
+      <updateRate>30</updateRate>
+      <leftJoint>mid_left_wheel_connect</leftJoint>
+      <rightJoint>mid_right_wheel_connect</rightJoint>
+      <wheelSeparation>0.23</wheelSeparation>
+      <wheelDiameter>0.08</wheelDiameter>
+      <wheelAcceleration>1</wheelAcceleration>
+      <wheelTorque>1</wheelTorque>
+      <rosDebugLevel>na</rosDebugLevel>
+    </plugin>
+  </gazebo>
+  <gazebo reference="base_scan">
+    <material>Gazebo/FlatBlack</material>
+    <sensor type="ray" name="lds_lfcd_sensor">
+      <pose>0 0 0 0 0 0</pose>
+      <visualize>$(arg laser_visual)</visualize>
+      <update_rate>5</update_rate>
+      <ray>
+        <scan>
+          <horizontal>
+            <samples>360</samples>
+            <resolution>1</resolution>
+            <min_angle>0.0</min_angle>
+            <max_angle>6.28319</max_angle>
+          </horizontal>
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